File: KiCad/SchoolDesk.sch (KiCad schematic (older format))
At the start: 15 parts, among them J1 Conn_1x5, J2 DIN-5_180degree, J3 Conn_1x1, J4 Conn_01x14_Female, J5 Conn_01x14_Female, J6 Conn_1x5

Commit message: First (untested) commit including PCB files.
Parts:
- removed C1: 10uF, C_SMD_3D:C_0805_2012Metric, symbol Device:CP1
- removed J1, J6: Conn_1x5, Pin_Headers:Pin_Header_Straight_1x05_Pitch2.00mm, symbol Connector:Conn_01x05_Female
- removed J3: Conn_1x1, P_2.54_3D:PinHeader_1x01_P2.54mm_Vertical, symbol Connector:Conn_01x01_Female
- removed R1, R3: R_FSR, Connectors:PJ320E_3.5mm_Jack, symbol Device:R_Variable
- removed RV1: 10k, Potentiometers:Potentiometer_Alps_RK09K_Vertical, symbol Device:R_POT
- added D1: LED_RCBG, LED_THT_3D:LED_D5.0mm-4_RGB, symbol Device:LED_RCBG
- added J1, J3, J9: 1x2, Pin_Headers:Pin_Header_Straight_1x02_Pitch2.00mm, symbol Connector:Conn_01x02_Female
- added J10, J11, J12: 1x1, Pin_Headers:Pin_Header_Straight_1x01_Pitch2.00mm, symbol Connector:Conn_01x01_Female
- added J13, J6, J7: AudioJack4, Conn_Aud_3D:Jack_3.5mm_PJ320D_Horizontal, symbol Connector:AudioJack4
- added J8: 1x02, Pin_Headers:Pin_Header_Straight_1x02_Pitch2.00mm, symbol Connector:Conn_01x02_Female
- added R1, R11: 10k, Resistors_ThroughHole:R_Axial_DIN0207_L6.3mm_D2.5mm_P2.54mm_Vertical, symbol Device:R
- added R10, R8, R9: 10k, R_SMD_3D:R_0805_2012Metric, symbol Device:R
- added R3: 330, R_SMD_3D:R_0805_2012Metric, symbol Device:R
- added SW1: Rotary_Encoder_Switch, digikey-footprints:Rotary_Encoder_Switched_PEC11R, symbol Device:Rotary_Encoder_Switch
- R2: value 10k -> 330; footprint Resistors_ThroughHole:R_Axial_DIN0207_L6.3mm_D2.5mm_P2.54mm_Vertical -> R_SMD_3D:R_0805_2012Metric
- R7: value 47k -> 330
Connections:
- net GND: now also J2.2, D1.2 (K), R1.1, R11.1, SW1.S1; no longer R2.1
- net at J4.7 (Pin_7): now also R4.2, J6.S; no longer R2.2
- net 3.3v: now reaches J4.3 (Pin_3), R5.1
- net 3.3v: now also J13.T, J6.T, J7.T, SW1.C
- net at J4.6 (Pin_6): now also J7.S, R1.2; no longer R4.2
- net at R7.1: now also D1.4 (GA)
- net at J4.13 (Pin_13): now also J13.S, R11.2; no longer R7.2
- net at J4.10 (Pin_10): now also J9.1 (Pin_1)
- net at J4.11 (Pin_11): now also J9.2 (Pin_2)
- net at J4.12 (Pin_12): now also J11.1 (Pin_1)
- net at J4.4 (Pin_4): now also J12.1 (Pin_1)
- net at J4.5 (Pin_5): now also J3.2 (Pin_2)
- net at J4.8 (Pin_8): now also J8.2 (Pin_2)
- net at J4.9 (Pin_9): now also J8.1 (Pin_1)
- net at J5.10 (Pin_10): now also R6.1; no longer R6.2
- net at J5.11 (Pin_11): now also R3.2
- net at J5.12 (Pin_12): now also R7.2
- net at J5.2 (Pin_2): now also J10.1 (Pin_1)
- net at J5.3 (Pin_3): now also J1.2 (Pin_2)
- net at J5.4 (Pin_4): now also R10.2
- net at J5.5 (Pin_5): now also J1.1 (Pin_1)
- net at J5.6 (Pin_6): now also J3.1 (Pin_1)
- net at J5.7 (Pin_7): now also R8.2
- net at J5.8 (Pin_8): now also R2.2
- net at J5.9 (Pin_9): now also R9.2
- net at J2.5: now also R6.2; no longer R6.1
- new net: R10.1, SW1.A
- new net: R8.1, SW1.B
- new net: R9.1, SW1.S2
- new net: D1.1 (RA), R2.1
- new net: D1.3 (BA), R3.1
- no-connect marks 14 -> 11
Other:
- moved on the sheet: J2, J4, J5, R4, R5, R6

Commit message: Add KiCad files
Parts:
- removed R10, R8, R9: 10k, R_SMD_3D:R_0805_2012Metric, symbol Device:R
- D1: footprint LED_THT_3D:LED_D5.0mm-4_RGB -> LED_SMD_3D:LED_RGB_1210
Connections:
- net 3.3v: no longer SW1.C
- net GND: now also SW1.C
- net at J5.11 (Pin_11): now also R7.2; no longer R3.2
- net at J5.12 (Pin_12): now also R3.2; no longer R7.2
- net at J5.4 (Pin_4): now also SW1.A
- net at J5.7 (Pin_7): now also SW1.B
- net at J5.9 (Pin_9): now also SW1.S2
Changed lines of the file:
@@
 	1    0    0    -1
 $EndComp
-Text GLabel 2800 2350 2    50   Input ~ 0
-3.3v
-$Comp
-L Device:R R8
-U 1 1 5E25E479
-P 3150 2450
-F 0 "R8" V 2943 2450 50  0000 C CNN
-F 1 "10k" V 3034 2450 50  0000 C CNN
-F 2 "R_SMD_3D:R_0805_2012Metric" V 3080 2450 50  0001 C CNN
-F 3 "~" H 3150 2450 50  0001 C CNN
-	1    3150 2450
-	0    -1   1    0
-$EndComp
-$Comp
-L Device:R R9
-U 1 1 5E2620CF
-P 2050 2450
-F 0 "R9" V 1843 2450 50  0000 C CNN
-F 1 "10k" V 1934 2450 50  0000 C CNN
-F 2 "R_SMD_3D:R_0805_2012Metric" V 1980 2450 50  0001 C CNN
-F 3 "~" H 2050 2450 50  0001 C CNN
-	1    2050 2450
-	0    1    -1   0
-$EndComp
-Wire Wire Line
-	3000 2450 2800 2450
 $Comp
 L Device:Rotary_Encoder_Switch SW1
@@
 	0    1    -1   0
 $EndComp
-$Comp
-L Device:R R10
-U 1 1 5E263249
-P 3150 2150
-F 0 "R10" V 2943 2150 50  0000 C CNN
-F 1 "10k" V 3034 2150 50  0000 C CNN
-F 2 "R_SMD_3D:R_0805_2012Metric" V 3080 2150 50  0001 C CNN
-F 3 "~" H 3150 2150 50  0001 C CNN
-	1    3150 2150
-	0    -1   1    0
-$EndComp
 Wire Wire Line
 	2200 2250 2050 2250
@@
 	4050 2050 4700 2050
 Wire Wire Line
-	4700 2450 3300 2450
-Wire Wire Line
-	4700 2150 3300 2150
-Wire Wire Line
 	3500 1700 3500 2350
 Wire Wire Line
@@
 Wire Wire Line
 	1650 3050 3100 3050
-Wire Wire Line
-	3000 2150 3000 2250
-Wire Wire Line
-	3000 2250 2800 2250
-Wire Wire Line
-	4700 2650 1900 2650
-Wire Wire Line
-	1900 2650 1900 2450
 Wire Wire Line
 	4600 3700 4700 3700
@@
 F 0 "D1" H 5200 3433 50  0000 C CNN
 F 1 "LED_RCBG" H 5200 3524 50  0000 C CNN
-F 2 "LED_THT_3D:LED_D5.0mm-4_RGB" H 5200 3850 50  0001 C CNN
+F 2 "LED_SMD_3D:LED_RGB_1210" H 5200 3850 50  0001 C CNN
 F 3 "~" H 5200 3850 50  0001 C CNN
 	1    5200 3900
 	-1   0    0    1
 $EndComp
-Wire Wire Line
-	4600 3700 4600 2850
-Wire Wire Line
-	4600 2850 4700 2850
-Wire Wire Line
-	4500 3900 4500 2950
-Wire Wire Line
-	4500 2950 4700 2950
 $Comp
 L Device:R R11
@@
 	7150 4750 6900 4750
 Connection ~ 7150 3550
+Wire Wire Line
+	2800 2450 4700 2450
+Wire Wire Line
+	4700 2150 3000 2150
+Wire Wire Line
+	3000 2150 3000 2250
+Wire Wire Line
+	3000 2250 2800 2250
+Wire Wire Line
+	4700 2650 2200 2650
+Wire Wire Line
+	2200 2650 2200 2450
+$Comp
+L power:GND #PWR0107
+U 1 1 5E547569
+P 2800 2350
+F 0 "#PWR0107" H 2800 2100 50  0001 C CNN
+F 1 "GND" V 2805 2222 50  0000 R CNN
+F 2 "" H 2800 2350 50  0001 C CNN
+F 3 "" H 2800 2350 50  0001 C CNN
+	1    2800 2350
+	0    -1   -1   0
+$EndComp
+Wire Wire Line
+	4700 2850 4500 2850
+Wire Wire Line
+	4500 2850 4500 3900
+Wire Wire Line
+	4600 3700 4600 2950
+Wire Wire Line
+	4600 2950 4700 2950
 $EndSCHEMATC
